File: pcb/USB To TTL adapter.kicad_sch (KiCad schematic)
At the start: 21 parts, among them J1 USB_B, U1 CH340G, U2 PC817, U3 PC817, Y1 12 MHz

Commit message: Update Schematic
Parts:
- removed D3: LED, LED_SMD:LED_0805_2012Metric, symbol Device:LED
- added Q1, Q2: (no value), symbol Transistor_BJT:BC817
- added R8: (no value), symbol Device:R
- D1, D2: value LED -> (none)
- J2: value (none) -> Conn_01x04
- R3: value 1K -> (none); footprint Resistor_SMD:R_0805_2012Metric -> (none)
- R4, R6: value (none) -> 1K
- R5: value (none) -> 330
- renumbered C4 to C2, C2 to C3, C3 to C4
Connections:
- net GND: now also R6.2, Q1.2 (E); no longer U3.3
- net GND1: now also R2.2, R5.2, Q2.2 (E); no longer U2.3
- net VCC: now also U3.4; no longer R2.1, R3.1, R5.1
- net VDD: now also D2.2 (A), U2.4; no longer R6.1
- net at D2.1 (K): now also R2.1; no longer R2.2
- net at R3.2: now also Q1.1 (B)
- net at U2.1: now also R4.2; no longer R5.2
- net V3: now reaches C5.1, U1.4 (V3)
- net at J2.3 (Pin_3): now also R8.2; no longer U3.2
- new net: Q1.3 (C), U2.2
- new net: J2.2 (Pin_2), R5.1, U2.3
- new net: R3.1, U1.2 (TXD)
- new net: R6.1, U1.3 (RXD), U3.3
- new net: Q2.1 (B), R8.1
- new net: Q2.3 (C), U3.2
Other:
- note added: "Capacitores de desacople"
- note added: "GND1"
- note added: "LED de estado PBP"
- note added: "LED de estado USB"
- note added: "RXD <- RX_iso"
- note added: "RX_iso"
- note added: "TXD -> TX_iso"
- note added: "TX_iso"
- note removed: "GND"
- note removed: "RX"
- note removed: "TX"
- company: Emiliano Eduardo Rodriguez -> Autor: Emiliano Eduardo Rodriguez
- title: USB To TTL isolated -> Réplica de USB To TTL isolated
- moved on the sheet: C1, C2, C3, C4, C5, D1, D2, J1, J2, R1, R2, R4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

Commit message: Update Schematic - PCB init
Parts:
- D1: value (none) -> LED GREEN
- D2: value (none) -> LED RED
- Q1, Q2: value (none) -> BC817; footprint (none) -> Package_TO_SOT_SMD:SOT-23
- R3, R6, R7, R8: footprint (none) -> Resistor_SMD:R_0805_2012Metric
- R4: value 1K -> (none); footprint (none) -> Resistor_SMD:R_0805_2012Metric
- R5: value 330 -> (none); footprint (none) -> Resistor_SMD:R_0805_2012Metric
- Y1: value 12 MHz -> (none); footprint Crystal:Crystal_HC49-U_Vertical -> (none)
Other:
- note added: "RX_iso = RX aislado"
- note added: "TX_iso = TX aislado"

Commit message: Diseño de PCB
Parts:
- R3, R8: value (none) -> 330K
- R4, R7: value (none) -> 1K8
- R5: value (none) -> 1K
- Y1: value (none) -> 12 MHz; footprint (none) -> Crystal:Crystal_HC49-4H_Vertical
Changed lines of the file:
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@@
+    (stroke (width 0) (type default) (color 0 0 0 0))
+  )
+  (polyline (pts (xy 106.68 71.12) (xy 106.68 90.17))
     (stroke (width 0) (type default) (color 0 0 0 0))
   )
@@
   )
   (wire (pts (xy 165.1 71.12) (xy 165.1 76.2))
+    (stroke (width 0) (type default) (color 0 0 0 0))
+  )
+  (polyline (pts (xy 106.68 90.17) (xy 113.03 90.17))
     (stroke (width 0) (type default) (color 0 0 0 0))
   )
@@
       (effects (font (size 1.27 1.27)) (justify left))
     )
-    (property "Value" "" (id 1) (at 167.64 68.5799 0)
+    (property "Value" "1K8" (id 1) (at 167.64 68.5799 0)
       (effects (font (size 1.27 1.27)) (justify left))
     )
@@
       (effects (font (size 1.27 1.27)) (justify left))
     )
-    (property "Value" "" (id 1) (at 185.42 125.7299 0)
+    (property "Value" "1K8" (id 1) (at 185.42 125.7299 0)
       (effects (font (size 1.27 1.27)) (justify left))
     )
@@
     (in_bom yes) (on_board yes) (fields_autoplaced)
     (property "Reference" "R3" (id 0) (at 151.13 83.82 90))
-    (property "Value" "" (id 1) (at 151.13 86.36 90))
+    (property "Value" "330K" (id 1) (at 151.13 86.36 90))
     (property "Footprint" "Resistor_SMD:R_0805_2012Metric" (id 2) (at 151.13 91.948 90)
       (effects (font (size 1.27 1.27)) hide)
@@
     (in_bom yes) (on_board yes) (fields_autoplaced)
     (property "Reference" "Y1" (id 0) (at 90.17 110.49 0))
-    (property "Value" "" (id 1) (at 90.17 113.03 0))
-    (property "Footprint" "" (id 2) (at 90.17 116.84 0)
+    (property "Value" "12 MHz" (id 1) (at 90.17 113.03 0))
+    (property "Footprint" "Crystal:Crystal_HC49-4H_Vertical" (id 2) (at 90.17 116.84 0)
       (effects (font (size 1.27 1.27)) hide)
     )
@@
       (effects (font (size 1.27 1.27)) (justify left))
     )
-    (property "Value" "" (id 1) (at 186.69 90.1699 0)
+    (property "Value" "1K" (id 1) (at 186.69 90.1699 0)
       (effects (font (size 1.27 1.27)) (justify left))
     )
@@
     (in_bom yes) (on_board yes) (fields_autoplaced)
     (property "Reference" "R8" (id 0) (at 196.85 137.16 90))
-    (property "Value" "" (id 1) (at 196.85 139.7 90))
+    (property "Value" "330K" (id 1) (at 196.85 139.7 90))
     (property "Footprint" "Resistor_SMD:R_0805_2012Metric" (id 2) (at 196.85 145.288 90)
       (effects (font (size 1.27 1.27)) hide)
