File: pcb/USB To TTL adapter.kicad_pcb (KiCad board)
At the start: 2 copper layers, 60 x 31 mm, 23 parts, among them J1 USB_B, J2 Conn_01x04, Q1 BC817, Q2 BC817, U1 CH340G, U2 PC817, U3 PC817, Y1 12 MHz

Commit message: Diseño de PCB
Parts:
- moved R6 16.7 mm to (152.5, 87.0), turned to 180 degrees
- moved R8 13.1 mm to (173.0, 96.4), turned to -90 degrees
- moved R3 12.0 mm to (148.0, 85.0), turned to 90 degrees
- moved Q2 8.49 mm to (168.0, 91.0), turned to 180 degrees
- moved R5 7.16 mm to (168.0, 81.5), turned to 90 degrees
- moved C2 6.52 mm to (136.5, 79.5), turned to 180 degrees
- moved C3 6.50 mm to (137.5, 98.0), turned to -90 degrees
- moved C4 6.50 mm to (132.5, 98.0), turned to -90 degrees
- moved R2 5.32 mm to (166.5, 74.0), turned to 180 degrees
- moved C5 5.02 mm to (136.5, 91.0), turned to 90 degrees
- moved Y1 4.95 mm to (142.0, 74.5), turned to -90 degrees
- moved C1 4.53 mm to (136.5, 74.5), turned to 180 degrees
- moved R7 4.27 mm to (164.0, 97.5)
- moved U1 3.58 mm to (144.9, 92.5)
- moved Q1 3.16 mm to (149.0, 77.0), turned to 90 degrees
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Routing:
- net VCC: track 0.00 -> 93.0 mm, vias 0 -> 2
- net GND: track 0.00 -> 87.3 mm, vias 0 -> 3
- net VDD: track 0.00 -> 64.6 mm, vias 0 -> 2
- net Net-(J1-Pad3): track 0.00 -> 24.2 mm, vias 0 -> 1
- net GND1: track 0.00 -> 24.2 mm, vias 0 -> 1
- net Net-(C1-Pad1): track 0.00 -> 20.6 mm
- net Net-(J2-Pad3): track 0.00 -> 19.6 mm, vias 0 -> 1
- net Net-(J1-Pad2): track 0.00 -> 17.7 mm, vias 0 -> 1
- net Net-(Q1-Pad3): track 0.00 -> 16.5 mm
- net Net-(C2-Pad1): track 0.00 -> 15.9 mm
- net Net-(J2-Pad2): track 0.00 -> 15.0 mm, vias 0 -> 1
- net Net-(R6-Pad1): track 0.00 -> 14.6 mm
- net /V3: track 0.00 -> 10.7 mm
- net Net-(Q2-Pad1): track 0.00 -> 7.00 mm
- net Net-(Q1-Pad1): track 0.00 -> 6.17 mm
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Other:
- board size 60 x 31 mm -> 65.5 x 31 mm
- board text added: "Emiliano Rodriguez - DCI - CESE"
- board text added: "USB To TTL Isolated"

Commit message: update PCB
Routing:
- net VCC: track 93.0 -> 96.0 mm
- added copper zone on F.Cu, net (none)
- added copper zone on B.Cu, net GND
- added copper zone on B.Cu, net GND1
Other:
- board text added: "USB To TTL Isolated v1.0"
- board text removed: "USB To TTL Isolated"
Changed lines of the file:
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@@
   )
   (paper "A4")
+  (title_block
+    (title "Réplica de USB To TTL isolated")
+    (date "2022-08-18")
+    (rev "v1.0")
+    (company "Autor: Emiliano Eduardo Rodriguez ")
+  )
   (layers
     (0 "F.Cu" signal)
@@
     (effects (font (size 2 1.5) (thickness 0.375)) (justify mirror))
   )
-  (gr_text "USB To TTL Isolated" (at 160 73) (layer "B.SilkS")
+  (gr_text "USB To TTL Isolated             v1.0" (at 148 73) (layer "B.SilkS")
     (effects (font (size 3 2) (thickness 0.5)) (justify mirror))
   )
-  (segment (start 143.699511 76.199511) (end 143.699511 82.020009) (width 0.7) (layer "F.Cu") (net 1))
+  (segment (start 143.699511 76.199511) (end 143.699511 82.020009) (width 0.6) (layer "F.Cu") (net 1))
   (segment (start 137.45 74.5) (end 142 74.5) (width 0.8) (layer "F.Cu") (net 1))
-  (segment (start 143.699511 82.020009) (end 141.71952 84) (width 0.7) (layer "F.Cu") (net 1))
-  (segment (start 141.71952 84) (end 141.71952 89) (width 0.7) (layer "F.Cu") (net 1))
-  (segment (start 142 74.5) (end 143.699511 76.199511) (width 0.7) (layer "F.Cu") (net 1))
+  (segment (start 143.699511 82.020009) (end 141.71952 84) (width 0.6) (layer "F.Cu") (net 1))
+  (segment (start 141.71952 84) (end 141.71952 89) (width 0.6) (layer "F.Cu") (net 1))
+  (segment (start 142 74.5) (end 143.699511 76.199511) (width 0.6) (layer "F.Cu") (net 1))
   (segment (start 128.5 94.5) (end 128.5 96.9125) (width 0.7) (layer "F.Cu") (net 2))
   (segment (start 135.978623 90.05) (end 131.528623 94.5) (width 0.7) (layer "F.Cu") (net 2))
@@
   (segment (start 141.88 79.5) (end 142 79.38) (width 0.8) (layer "F.Cu") (net 3))
   (segment (start 149.31 96.250916) (end 149.31 94.95) (width 0.7) (layer "F.Cu") (net 4))
-  (segment (start 155.19 93.81) (end 152 97) (width 0.7) (layer "F.Cu") (net 4))
   (segment (start 139.5 98) (end 147.560916 98) (width 0.7) (layer "F.Cu") (net 4))
   (segment (start 134.928143 72.70048) (end 132.837011 74.791612) (width 0.7) (layer "F.Cu") (net 4))
@@
   (segment (start 147.560916 98) (end 149.31 96.250916) (width 0.7) (layer "F.Cu") (net 4))
   (segment (start 134.95 97.05) (end 137.5 97.05) (width 0.7) (layer "F.Cu") (net 4))
-  (segment (start 152 97) (end 150.059084 97) (width 0.7) (layer "F.Cu") (net 4))
   (segment (start 152.78798 72.70048) (end 134.928143 72.70048) (width 0.7) (layer "F.Cu") (net 4))
   (segment (start 125.288614 88.250489) (end 129.750489 88.250489) (width 0.7) (layer "F.Cu") (net 4))
   (segment (start 132.837011 74.791612) (end 132.837011 84.700489) (width 0.7) (layer "F.Cu") (net 4))
-  (segment (start 150.059084 97) (end 149.31 96.250916) (width 0.7) (layer "F.Cu") (net 4))
-  (segment (start 155.19 93.27) (end 155.19 93.81) (width 0.7) (layer "F.Cu") (net 4))
+  (segment (start 153 98) (end 147.560916 98) (width 0.7) (layer "F.Cu") (net 4))
+  (segment (start 155.19 93.27) (end 155.19 95.81) (width 0.7) (layer "F.Cu") (net 4))
   (segment (start 138.55 97.05) (end 139.5 98) (width 0.7) (layer "F.Cu") (net 4))
   (segment (start 129.750489 88.250489) (end 131.2875 89.7875) (width 0.7) (layer "F.Cu") (net 4))
+  (segment (start 155.19 95.81) (end 153 98) (width 0.7) (layer "F.Cu") (net 4))
   (via (at 134.95 97.05) (size 0.8) (drill 0.4) (layers "F.Cu" "B.Cu") (net 4))
   (via (at 131.2875 89.7875) (size 0.8) (drill 0.4) (layers "F.Cu" "B.Cu") (net 4))
@@
   (segment (start 168 76.5) (end 166 78.5) (width 0.7) (layer "B.Cu") (net 8))
   (segment (start 175.5 77.5) (end 174 79) (width 0.8) (layer "B.Cu") (net 8))
-  (segment (start 143.5 86.5) (end 143.5 85.5) (width 0.5) (layer "F.Cu") (net 9))
-  (segment (start 142.96 90) (end 142.96 87.04) (width 0.5) (layer "F.Cu") (net 9))
-  (segment (start 142.96 87.04) (end 143.5 86.5) (width 0.5) (layer "F.Cu") (net 9))
+  (segment (start 143.5 86.5) (end 143.5 85.5) (width 0.6) (layer "F.Cu") (net 9))
+  (segment (start 142.96 90) (end 142.96 87.04) (width 0.59) (layer "F.Cu") (net 9))
+  (segment (start 142.96 87.04) (end 143.5 86.5) (width 0.59) (layer "F.Cu") (net 9))
   (via (at 143.5 85.5) (size 0.8) (drill 0.4) (layers "F.Cu" "B.Cu") (net 9))
   (segment (start 137.5 85.5) (end 143.5 85.5) (width 0.7) (layer "B.Cu") (net 9))
   (segment (start 131.2875 83.75) (end 135.75 83.75) (width 0.7) (layer "B.Cu") (net 9))
   (segment (start 135.75 83.75) (end 137.5 85.5) (width 0.7) (layer "B.Cu") (net 9))
-  (segment (start 144.23 87.77) (end 144.23 90) (width 0.5) (layer "F.Cu") (net 10))
-  (segment (start 145 87) (end 144.23 87.77) (width 0.5) (layer "F.Cu") (net 10))
-  (segment (start 145 84) (end 145 87) (width 0.5) (layer "F.Cu") (net 10))
+  (segment (start 144.23 87.77) (end 144.23 90) (width 0.6) (layer "F.Cu") (net 10))
+  (segment (start 145 87) (end 144.23 87.77) (width 0.6) (layer "F.Cu") (net 10))
+  (segment (start 145 84) (end 145 87) (width 0.6) (layer "F.Cu") (net 10))
   (via (at 145 84) (size 0.8) (drill 0.4) (layers "F.Cu" "B.Cu") (net 10))
   (segment (start 136.5 82) (end 138.5 84) (width 0.7) (layer "B.Cu") (net 10))
@@
   (segment (start 162.81 93.27) (end 162.81 97.2225) (width 0.7) (layer "F.Cu") (net 21))
   (segment (start 162.81 97.2225) (end 163.0875 97.5) (width 0.7) (layer "F.Cu") (net 21))
+  (zone (net 0) (net_name "") (layer "F.Cu") (hatch edge 0.508)
+    (connect_pads (clearance 0.508))
+    (min_thickness 0.254) (filled_areas_thickness no)
+    (fill yes (thermal_gap 0.508) (thermal_bridge_width 0.508))
+    (polygon
+      (pts
+        (xy 156.5 105.5)
+        (xy 110 105.5)
+        (xy 110 65)
+        (xy 156.5 65)
+      )
+    )
+  )
+  (zone (net 0) (net_name "") (layer "F.Cu") (hatch edge 0.508)
+    (connect_pads (clearance 0.508))
+    (min_thickness 0.254) (filled_areas_thickness no)
+    (fill yes (thermal_gap 0.508) (thermal_bridge_width 0.508))
+    (polygon
+      (pts
+        (xy 184.5 105)
+        (xy 161.5 105)
+        (xy 161.5 65)
+        (xy 184.5 65)
+      )
+    )
+  )
+  (zone (net 13) (net_name "GND1") (layer "B.Cu") (hatch edge 0.508)
+    (connect_pads (clearance 0.508))
+    (min_thickness 0.254) (filled_areas_thickness no)
+    (fill yes (thermal_gap 0.508) (thermal_bridge_width 0.508))
+    (polygon
+      (pts
+        (xy 182.5 102.5)
+        (xy 161.5 102.5)
+        (xy 161.5 68)
+        (xy 182.5 68)
+      )
+    )
+  )
+  (zone (net 2) (net_name "GND") (layer "B.Cu") (hatch edge 0.508)
+    (connect_pads (clearance 0.508))
+    (min_thickness 0.254) (filled_areas_thickness no)
+    (fill yes (thermal_gap 0.508) (thermal_bridge_width 0.508))
+    (polygon
+      (pts
+        (xy 156.5 102.5)
+        (xy 112.5 102.5)
+        (xy 112.5 68)
+        (xy 156.5 68)
+      )
+    )
+  )
 )
